File: Seadream Avionics Barney/Seadream Avionics Barney.kicad_pcb (KiCad board)
At the start: 2 copper layers, 26 x 63 mm, 41 parts, among them J1 B2B-PH-K-S(LF)(SN), J2 C393939, J3 B2B-PH-K-S(LF)(SN), SW1 SSSS810701, U1 BMP280, U2 ESP32-S3-MINI-1U-N8, U3 LSM6DSO32TR, U4 LD1117S33TR, U5 SHT40-AD1B-R3, U6 LD39200PU33R, U7 MAX98357AETE_T

Commit message: Updated PCB files
Connections:
- net Net-(J3-Pin_1) renamed /OUT+
- net Net-(J3-Pin_2) renamed /OUT-
Other:
- board text added: "B"
- board text added: "GND 3.7V"
- board text added: "OUT- OUT+"
- board text added: "R"
Changed lines of the file:
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@@
 	(net 13 "Net-(J2-CC1)")
 	(net 14 "Net-(J2-CC2)")
-	(net 15 "Net-(J3-Pin_2)")
-	(net 16 "Net-(J3-Pin_1)")
+	(net 15 "/OUT+")
+	(net 16 "/OUT-")
 	(net 17 "/MOSI")
 	(net 18 "unconnected-(MICRO_SD1-DAT2-Pad1)")
@@
 			(layers "F.Cu" "F.Mask" "F.Paste")
 			(roundrect_rratio 0.125)
-			(net 16 "Net-(J3-Pin_1)")
+			(net 15 "/OUT+")
 			(pinfunction "OUTP")
 			(pintype "output")
@@
 			(layers "F.Cu" "F.Mask" "F.Paste")
 			(roundrect_rratio 0.125)
-			(net 15 "Net-(J3-Pin_2)")
+			(net 16 "/OUT-")
 			(pinfunction "OUTN")
 			(pintype "output")
@@
 			(remove_unused_layers no)
 			(roundrect_rratio 0.208333)
-			(net 16 "Net-(J3-Pin_1)")
+			(net 15 "/OUT+")
 			(pinfunction "Pin_1")
 			(pintype "passive")
@@
 			(layers "*.Cu" "*.Mask")
 			(remove_unused_layers no)
-			(net 15 "Net-(J3-Pin_2)")
+			(net 16 "/OUT-")
 			(pinfunction "Pin_2")
 			(pintype "passive")
@@
 	(gr_circle
 		(center 143.5 41.25)
-		(end 143.5 39)
-		(stroke
-			(width 0.05)
-			(type solid)
-		)
-		(fill no)
-		(layer "Dwgs.User")
-	)
-	(gr_circle
-		(center 164.5 58.75)
-		(end 164.5 56.5)
-		(stroke
-			(width 0.05)
-			(type solid)
-		)
-		(fill no)
-		(layer "Dwgs.User")
-	)
-	(gr_circle
-		(center 164.5 99.25)
-		(end 164.5 97)
-		(stroke
-			(width 0.05)
-			(type solid)
-		)
-		(fill no)
-		(layer "Dwgs.User")
-	)
-	(gr_circle
-		(center 143.5 99.25)
-		(end 143.5 97)
-		(stroke
-			(width 0.05)
-			(type solid)
-		)
-		(fill no)
-		(layer "Dwgs.User")
-	)
-	(gr_circle
-		(center 143.5 41.25)
 		(end 143.5 40.25)
 		(stroke
 			(width 0.05)
-			(type default)
+			(type solid)
 		)
 		(fill no)
@@
 	(gr_circle
 		(center 164.5 99.25)
-		(end 164.5 98.25)
+		(end 165.5 99.25)
 		(stroke
 			(width 0.05)
-			(type default)
+			(type solid)
 		)
 		(fill no)
@@
 		(layer "Edge.Cuts")
 	)
+	(gr_text "B"
+		(at 165.5 67.75 0)
+		(layer "F.SilkS")
+		(effects
+			(font
+				(size 1 1)
+				(thickness 0.2)
+				(bold yes)
+			)
+			(justify left bottom)
+		)
+	)
+	(gr_text "R"
+		(at 165.5 63.25 0)
+		(layer "F.SilkS")
+		(effects
+			(font
+				(size 1 1)
+				(thickness 0.2)
+				(bold yes)
+			)
+			(justify left bottom)
+		)
+	)
+	(gr_text "GND\n3.7V"
+		(at 149.75 49 0)
+		(layer "B.SilkS")
+		(effects
+			(font
+				(size 1 1)
+				(thickness 0.2)
+				(bold yes)
+			)
+			(justify left bottom mirror)
+		)
+	)
+	(gr_text "OUT-\nOUT+"
+		(at 146.5 65 90)
+		(layer "B.SilkS")
+		(effects
+			(font
+				(size 1 1)
+				(thickness 0.2)
+				(bold yes)
+			)
+			(justify left bottom mirror)
+		)
+	)
 	(segment
 		(start 160.5 89.75)
@@
 	)
 	(segment
-		(start 143.344 71.156)
-		(end 144 70.5)
+		(start 144.065 72.435)
+		(end 146 70.5)
 		(width 0.2)
 		(layer "F.Cu")
@@
 	)
 	(segment
-		(start 143.603158 80.45)
-		(end 143.344 80.190842)
+		(start 144.065 79.95)
+		(end 144.065 72.435)
 		(width 0.2)
 		(layer "F.Cu")
@@
 	)
 	(segment
-		(start 143.344 80.190842)
-		(end 143.344 71.156)
+		(start 143.344 71.156)
+		(end 144 70.5)
 		(width 0.2)
 		(layer "F.Cu")
-		(net 15)
+		(net 16)
 	)
 	(segment
-		(start 144.065 80.45)
-		(end 143.603158 80.45)
+		(start 143.603158 80.45)
+		(end 143.344 80.190842)
 		(width 0.2)
 		(layer "F.Cu")
-		(net 15)
+		(net 16)
 	)
 	(segment
-		(start 144.065 72.435)
-		(end 146 70.5)
+		(start 143.344 80.190842)
+		(end 143.344 71.156)
 		(width 0.2)
 		(layer "F.Cu")
@@
 	)
 	(segment
-		(start 144.065 79.95)
-		(end 144.065 72.435)
+		(start 144.065 80.45)
+		(end 143.603158 80.45)
 		(width 0.2)
 		(layer "F.Cu")
@@
 			)
 		)
+	)
+	(zone
+		(net 0)
+		(net_name "")
+		(layers "F.Cu" "B.Cu")
+		(hatch edge 0.5)
+		(connect_pads
+			(clearance 0)
+		)
+		(min_thickness 0.25)
+		(filled_areas_thickness no)
+		(keepout
+			(tracks not_allowed)
+			(vias not_allowed)
+			(pads not_allowed)
+			(copperpour not_allowed)
+			(footprints not_allowed)
+		)
+		(placement
+			(enabled no)
+			(sheetname "/")
+		)
+		(fill
+			(thermal_gap 0.5)
+			(thermal_bridge_width 0.5)
+		)
+		(polygon
+			(pts
+				(arc
+					(start 162.25 58.75)
+					(mid 166.75 58.75)
+					(end 162.25 58.75)
+				)
+			)
+		)
+	)
+	(zone
+		(net 0)
+		(net_name "")
+		(layers "F.Cu" "B.Cu")
+		(hatch edge 0.5)
+		(connect_pads
+			(clearance 0)
+		)
+		(min_thickness 0.25)
+		(filled_areas_thickness no)
+		(keepout
+			(tracks not_allowed)
+			(vias not_allowed)
+			(pads not_allowed)
+			(copperpour not_allowed)
+			(footprints not_allowed)
+		)
+		(placement
+			(enabled no)
+			(sheetname "/")
+		)
+		(fill
+			(thermal_gap 0.5)
+			(thermal_bridge_width 0.5)
+		)
+		(polygon
+			(pts
+				(arc
+					(start 141.25 41.25)
+					(mid 145.75 41.25)
+					(end 141.25 41.25)
+				)
+			)
+		)
+	)
+	(zone
+		(net 0)
+		(net_name "")
+		(layers "F.Cu" "B.Cu")
+		(hatch edge 0.5)
+		(connect_pads
+			(clearance 0)
+		)
+		(min_thickness 0.25)
+		(filled_areas_thickness no)
+		(keepout
+			(tracks not_allowed)
+			(vias not_allowed)
+			(pads not_allowed)
+			(copperpour not_allowed)
+			(footprints not_allowed)
+		)
+		(placement
+			(enabled no)
+			(sheetname "/")
+		)
+		(fill
+			(thermal_gap 0.5)
+			(thermal_bridge_width 0.5)
+		)
+		(polygon
+			(pts
+				(arc
+					(start 162.25 99.25)
+					(mid 166.75 99.25)
+					(end 162.25 99.25)
+				)
+			)
+		)
+	)
+	(zone
+		(net 0)
+		(net_name "")
+		(layers "F.Cu" "B.Cu")
+		(hatch edge 0.5)
+		(connect_pads
+			(clearance 0)
+		)
+		(min_thickness 0.25)
+		(filled_areas_thickness no)
+		(keepout
+			(tracks not_allowed)
+			(vias not_allowed)
+			(pads not_allowed)
+			(copperpour not_allowed)
+			(footprints not_allowed)
+		)
+		(placement
+			(enabled no)
+			(sheetname "/")
+		)
+		(fill
+			(thermal_gap 0.5)
+			(thermal_bridge_width 0.5)
+		)
+		(polygon
+			(pts
+				(arc
+					(start 141.25 99.25)
+					(mid 145.75 99.25)
+					(end 141.25 99.25)
+				)
+			)
+		)
