File: Seadream Avionics Barney/Seadream Avionics Barney.kicad_sch (KiCad schematic)
At the start: 41 parts, among them J1 B2B-PH-K-S(LF)(SN), J2 C393939, J3 B2B-PH-K-S(LF)(SN), SW1 SSSS810701, U1 BMP280, U2 ESP32-S3-MINI-1U-N8, U3 LSM6DSO32TR, U4 LD1117S33TR, U5 SHT40-AD1B-R3, U6 LD39200PU33R, U7 MAX98357AETE_T

Commit message: Updated PCB files
Connections:
- net OUT-: now reaches J3.2 (Pin_2), U7.10 (OUTN)
- net OUT+: now reaches J3.1 (Pin_1), U7.9 (OUTP)
Other:
- moved on the sheet: J3
Changed lines of the file:
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@@
 	(wire
 		(pts
+			(xy 69.85 170.18) (xy 64.77 170.18)
+		)
+		(stroke
+			(width 0)
+			(type default)
+		)
+	)
+	(wire
+		(pts
 			(xy 139.7 80.01) (xy 149.86 80.01)
 		)
@@
 	(wire
 		(pts
+			(xy 69.85 167.64) (xy 64.77 167.64)
+		)
+		(stroke
+			(width 0)
+			(type default)
+		)
+	)
+	(wire
+		(pts
 			(xy 72.39 24.13) (xy 78.74 24.13)
 		)
@@
 		)
 	)
+	(label "OUT+"
+		(at 64.77 170.18 0)
+		(effects
+			(font
+				(size 1.27 1.27)
+			)
+			(justify left bottom)
+		)
+	)
+	(label "OUT-"
+		(at 64.77 167.64 0)
+		(effects
+			(font
+				(size 1.27 1.27)
+			)
+			(justify left bottom)
+		)
+	)
 	(label "D-"
 		(at 69.85 123.19 0)
@@
 	(symbol
 		(lib_id "Connector:Conn_01x02_Socket")
-		(at 69.85 170.18 0)
+		(at 74.93 170.18 0)
 		(mirror x)
 		(unit 1)
@@
 		(dnp no)
 		(property "Reference" "J3"
-			(at 71.882 167.894 0)
+			(at 76.962 167.894 0)
 			(effects
 				(font
@@
 		)
 		(property "Value" "B2B-PH-K-S(LF)(SN)"
-			(at 71.374 172.466 0)
+			(at 76.454 172.466 0)
 			(effects
 				(font
@@
 		)
 		(property "Footprint" "Connector_JST:JST_PH_B2B-PH-K_1x02_P2.00mm_Vertical"
-			(at 69.85 170.18 0)
+			(at 74.93 170.18 0)
 			(effects
 				(font
@@
 		)
 		(property "Datasheet" "~"
-			(at 69.85 170.18 0)
+			(at 74.93 170.18 0)
 			(effects
 				(font
@@
 		)
 		(property "Description" "Generic connector, single row, 01x02, script generated"
-			(at 69.85 170.18 0)
+			(at 74.93 170.18 0)
 			(effects
 				(font
