File: Seadream Avionics PCB/Seadream Avionics PCB.kicad_pcb (KiCad board)
At the start: 2 copper layers, 26 x 63 mm, 42 parts, among them J1 B2B-PH-K-S(LF)(SN), J2 C393939, J3 B2B-PH-K-S(LF)(SN), SW1 SSSS810701, U1 BMP280, U2 ESP32-S3-MINI-1U-N8, U3 LSM6DSO32TR, U4 LD1117S33TR, U5 SHT40-AD1B-R3, U6 LD39200PU33R, U7 MAX98357AETE_T

Commit message: IDK
Parts:
- J2: value C393939 -> TYPE-C16PIN; footprint TYPE-C_16PIN_2MD__073_:SHOUHAN_TYPE-C_16PIN_2MD__073_ -> 2FOOTPRINTS:SHOUHAN_TYPE-C_16PIN_2MD__073_
- MICRO_SD1: value C91145 -> TF-01A
Connections:
- U1 pad 5: unconnected-(U1-SDO-Pad5) -> GND
- U2 pad 61: GND -> (no net)
- U7 pad 4: GND -> +3.3V
Routing:
- net +3.3V: track 184.9 -> 186.3 mm
- net GND: track 156.1 -> 155.4 mm, vias 66 -> 65
