File: Seadream Avionics PCB/Seadream Avionics PCB.kicad_sch (KiCad schematic)
At the start: 41 parts, among them J1 B2B-PH-K-S(LF)(SN), J2 TYPE-C16PIN, J3 B2B-PH-K-S(LF)(SN), SW1 SSSS810701, U1 BMP280, U2 ESP32-S3-MINI-1U-N8, U3 LSM6DSO32TR, U4 LD1117S33TR, U5 SHT40-AD1B-R3, U6 LD39200PU33R, U7 MAX98357AETE_T

Commit message: IDK
Connections:
- net +3.3V: now also U7.4 (SD_MODE)
- net GND: now also U1.5 (SDO); no longer U7.4 (SD_MODE)
- no-connect marks 36 -> 35
Changed lines of the file:
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@@
 	)
 	(junction
+		(at 20.32 172.72)
+		(diameter 0)
+		(color 0 0 0 0)
+	)
+	(junction
 		(at 72.39 24.13)
 		(diameter 0)
@@
 	)
 	(no_connect
-		(at 232.41 27.94)
-	)
-	(no_connect
 		(at 69.85 29.21)
 	)
@@
 	(wire
 		(pts
+			(xy 227.33 30.48) (xy 227.33 27.94)
+		)
+		(stroke
+			(width 0)
+			(type default)
+		)
+	)
+	(wire
+		(pts
 			(xy 78.74 53.34) (xy 82.55 53.34)
 		)
@@
 	(wire
 		(pts
-			(xy 26.67 179.07) (xy 26.67 177.8)
-		)
-		(stroke
-			(width 0)
-			(type default)
-		)
-	)
-	(wire
-		(pts
 			(xy 114.3 40.64) (xy 119.38 40.64)
 		)
@@
 	(wire
 		(pts
-			(xy 19.05 172.72) (xy 29.21 172.72)
+			(xy 19.05 172.72) (xy 20.32 172.72)
 		)
 		(stroke
@@
 	(wire
 		(pts
-			(xy 26.67 177.8) (xy 29.21 177.8)
+			(xy 91.44 43.18) (xy 86.36 43.18)
 		)
 		(stroke
@@
 	(wire
 		(pts
-			(xy 91.44 43.18) (xy 86.36 43.18)
+			(xy 115.57 166.37) (xy 114.3 166.37)
 		)
 		(stroke
@@
 	(wire
 		(pts
-			(xy 115.57 166.37) (xy 114.3 166.37)
+			(xy 20.32 177.8) (xy 20.32 172.72)
 		)
 		(stroke
@@
 	(wire
 		(pts
+			(xy 20.32 172.72) (xy 29.21 172.72)
+		)
+		(stroke
+			(width 0)
+			(type default)
+		)
+	)
+	(wire
+		(pts
 			(xy 261.62 35.56) (xy 261.62 36.83)
 		)
@@
 	(wire
 		(pts
+			(xy 227.33 27.94) (xy 232.41 27.94)
+		)
+		(stroke
+			(width 0)
+			(type default)
+		)
+	)
+	(wire
+		(pts
 			(xy 218.44 77.47) (xy 226.06 77.47)
 		)
@@
 	(wire
 		(pts
+			(xy 20.32 177.8) (xy 29.21 177.8)
+		)
+		(stroke
+			(width 0)
+			(type default)
+		)
+	)
+	(wire
+		(pts
 			(xy 261.62 64.77) (xy 264.16 64.77)
 		)
@@
 	)
 	(symbol
+		(lib_id "power:GND")
+		(at 229.87 38.1 0)
+		(unit 1)
+		(exclude_from_sim no)
+		(in_bom yes)
+		(on_board yes)
+		(dnp no)
+		(fields_autoplaced yes)
+		(property "Reference" "#PWR036"
+			(at 229.87 44.45 0)
+			(effects
+				(font
+					(size 1.27 1.27)
+				)
+				(hide yes)
+			)
+		)
+		(property "Value" "GND"
+			(at 229.87 43.18 0)
+			(effects
+				(font
+					(size 1.27 1.27)
+				)
+			)
+		)
+		(property "Footprint" ""
+			(at 229.87 38.1 0)
+			(effects
+				(font
+					(size 1.27 1.27)
+				)
+				(hide yes)
+			)
+		)
+		(property "Datasheet" ""
+			(at 229.87 38.1 0)
+			(effects
+				(font
+					(size 1.27 1.27)
+				)
+				(hide yes)
+			)
+		)
+		(property "Description" "Power symbol creates a global label with name \"GND\" , ground"
+			(at 229.87 38.1 0)
+			(effects
+				(font
+					(size 1.27 1.27)
+				)
+				(hide yes)
+			)
+		)
+		(pin "1"
+		)
+		(instances
+			(project "Seadream Avionics PCB"
+				(path "/3eab51f1-e840-4fcb-ae14-6a5e4ec9e628"
+					(reference "#PWR036")
+					(unit 1)
+				)
+			)
+		)
+	)
+	(symbol
 		(lib_id "power:+3.3V")
 		(at 195.58 115.57 0)
@@
 	)
 	(symbol
+		(lib_id "power:GND")
+		(at 227.33 30.48 0)
+		(unit 1)
+		(exclude_from_sim no)
+		(in_bom yes)
+		(on_board yes)
+		(dnp no)
+		(fields_autoplaced yes)
+		(property "Reference" "#PWR040"
+			(at 227.33 36.83 0)
+			(effects
+				(font
+					(size 1.27 1.27)
+				)
+				(hide yes)
+			)
+		)
+		(property "Value" "GND"
+			(at 227.33 35.56 0)
+			(effects
+				(font
+					(size 1.27 1.27)
+				)
+			)
+		)
+		(property "Footprint" ""
+			(at 227.33 30.48 0)
+			(effects
+				(font
+					(size 1.27 1.27)
+				)
+				(hide yes)
+			)
+		)
+		(property "Datasheet" ""
+			(at 227.33 30.48 0)
+			(effects
+				(font
+					(size 1.27 1.27)
+				)
+				(hide yes)
+			)
+		)
+		(property "Description" "Power symbol creates a global label with name \"GND\" , ground"
+			(at 227.33 30.48 0)
+			(effects
+				(font
+					(size 1.27 1.27)
+				)
+				(hide yes)
+			)
+		)
+		(pin "1"
+		)
+		(instances
+			(project "Seadream Avionics PCB"
+				(path "/3eab51f1-e840-4fcb-ae14-6a5e4ec9e628"
+					(reference "#PWR040")
+					(unit 1)
+				)
+			)
+		)
+	)
+	(symbol
 		(lib_id "Device:R")
 		(at 104.14 177.8 0)
@@
 					(unit 1)
 				)
-			)
-		)
-	)
-	(symbol
-		(lib_id "power:GND")
-		(at 26.67 179.07 0)
-		(unit 1)
-		(exclude_from_sim no)
-		(in_bom yes)
-		(on_board yes)
-		(dnp no)
-		(fields_autoplaced yes)
-		(property "Reference" "#PWR036"
-			(at 26.67 185.42 0)
-			(effects
-				(font
-					(size 1.27 1.27)
-				)
-				(hide yes)
-			)
-		)
-		(property "Value" "GND"
-			(at 26.67 184.15 0)
-			(effects
-				(font
-					(size 1.27 1.27)
-				)
-			)
-		)
-		(property "Footprint" ""
-			(at 26.67 179.07 0)
-			(effects
-				(font
-					(size 1.27 1.27)
-				)
-				(hide yes)
-			)
-		)
-		(property "Datasheet" ""
-			(at 26.67 179.07 0)
-			(effects
-				(font
-					(size 1.27 1.27)
-				)
-				(hide yes)
-			)
-		)
-		(property "Description" "Power symbol creates a global label with name \"GND\" , ground"
-			(at 26.67 179.07 0)
-			(effects
-				(font
-					(size 1.27 1.27)
-				)
-				(hide yes)
-			)
-		)
-		(pin "1"
-		)
-		(instances
-			(project "Seadream Avionics Barney"
-				(path "/3eab51f1-e840-4fcb-ae14-6a5e4ec9e628"
-					(reference "#PWR036")
-					(unit 1)
-				)
